File: Hardware/Week 2/Schematics/KiCad/fireworks.kicad_sch (KiCad schematic)
At the start: 0 parts

Commit message: Finish the schematic
Parts:
- added C1, C10, C11, C12, C13, C14, C15, C16, C17, C18, C19, C2, C20, C21, C22, C23, C24, C3, C4, C5, C6, C7, C8, C9: 10u, symbol Device:C
- added D1, D10, D11, D12, D13, D14, D15, D16, D17, D18, D19, D2, D20, D21, D22, D23, D24, D25, D26, D27, D28, D29, D3, D30, D4, D5, D6, D7, D8, D9: LED, symbol Device:LED
- added Q1, Q10, Q11, Q12, Q13, Q14, Q15, Q16, Q17, Q18, Q19, Q2, Q20, Q21, Q22, Q23, Q24, Q25, Q26, Q27, Q28, Q29, Q3, Q30, Q4, Q5, Q6, Q7, Q8, Q9: NPN, symbol Simulation_SPICE:NPN
- added R1, R10, R11, R12, R13, R14, R15, R16, R17, R18, R19, R2, R20, R21, R22, R23, R24, R25, R26, R27, R28, R29, R3, R30, R4, R5, R6, R7, R8, R9: 1K, symbol Device:R
- added SW1: SW_Push, symbol Switch:SW_Push
Connections:
- new net: R1.1, R10.1, R11.1, R12.1, R13.1, R14.1, R15.1, R16.1, R17.1, R18.1, R19.1, R2.1, R20.1, R21.1, R22.1, R23.1, R24.1, R25.1, R26.1, R27.1, R28.1, R29.1, R3.1, R30.1, R4.1, R5.1, R6.1, R7.1, R8.1, R9.1, SW1.2
- new net: Q30.1 (C), R30.2
- new net: D29.2 (A), Q29.3 (E)
- new net: Q17.1 (C), R17.2
- new net: C13.1, Q17.2 (B)
- new net: D17.2 (A), Q17.3 (E)
- new net: Q4.1 (C), R4.2
- new net: C3.1, Q4.2 (B)
- new net: D4.2 (A), Q4.3 (E)
- new net: Q1.1 (C), R1.2
- new net: C1.2, C2.2, C3.2, C4.2, Q1.2 (B)
- new net: D1.2 (A), Q1.3 (E)
- new net: C24.1, Q30.2 (B)
- new net: C21.2, C22.2, C23.2, C24.2, Q26.2 (B)
- new net: Q28.1 (C), R28.2
- new net: C22.1, Q28.2 (B)
- new net: D28.2 (A), Q28.3 (E)
- new net: Q12.1 (C), R12.2
- new net: C2.1, Q3.2 (B)
- new net: Q25.1 (C), R25.2
- new net: C20.1, Q25.2 (B)
- new net: D25.2 (A), Q25.3 (E)
- new net: Q7.1 (C), R7.2
- new net: Q26.1 (C), R26.2
- new net: Q19.1 (C), R19.2
- new net: D8.2 (A), Q8.3 (E)
- new net: Q27.1 (C), R27.2
- new net: C21.1, Q27.2 (B)
- new net: D27.2 (A), Q27.3 (E)
- new net: C1.1, Q2.2 (B)
- new net: D19.2 (A), Q19.3 (E)
- new net: Q23.1 (C), R23.2
- new net: C18.1, Q23.2 (B)
- new net: D23.2 (A), Q23.3 (E)
- new net: C5.1, Q7.2 (B)
- new net: D7.2 (A), Q7.3 (E)
- new net: D11.2 (A), Q11.3 (E)
- new net: Q9.1 (C), R9.2
- new net: C7.1, Q9.2 (B)
- new net: D9.2 (A), Q9.3 (E)
- new net: Q13.1 (C), R13.2
- new net: C10.1, Q13.2 (B)
- new net: D13.2 (A), Q13.3 (E)
- new net: C5.2, C6.2, C7.2, C8.2, Q6.2 (B)
- new net: Q16.1 (C), R16.2
- new net: C16.1, Q20.2 (B)
- new net: C13.2, C14.2, C15.2, C16.2, Q16.2 (B)
- new net: Q14.1 (C), R14.2
- new net: C11.1, Q14.2 (B)
- new net: D14.2 (A), Q14.3 (E)
- new net: C10.2, C11.2, C12.2, C9.2, Q11.2 (B)
- new net: C6.1, Q8.2 (B)
- new net: Q5.1 (C), R5.2
- new net: C9.1, Q12.2 (B)
- new net: D12.2 (A), Q12.3 (E)
- new net: D30.2 (A), Q30.3 (E)
- new net: Q22.1 (C), R22.2
- new net: C17.1, Q22.2 (B)
- new net: D22.2 (A), Q22.3 (E)
- new net: Q20.1 (C), R20.2
- new net: D20.2 (A), Q20.3 (E)
- new net: Q15.1 (C), R15.2
- new net: C12.1, Q15.2 (B)
- new net: D15.2 (A), Q15.3 (E)
- new net: Q2.1 (C), R2.2
- new net: D2.2 (A), Q2.3 (E)
- new net: C19.1, Q24.2 (B)
- new net: C17.2, C18.2, C19.2, C20.2, Q21.2 (B)
- new net: C23.1, Q29.2 (B)
- new net: Q6.1 (C), R6.2
- new net: D6.2 (A), Q6.3 (E)
- new net: C14.1, Q18.2 (B)
- new net: Q10.1 (C), R10.2
- new net: D24.2 (A), Q24.3 (E)
- new net: D26.2 (A), Q26.3 (E)
- new net: C15.1, Q19.2 (B)
- new net: Q24.1 (C), R24.2
- new net: D16.2 (A), Q16.3 (E)
- new net: Q3.1 (C), R3.2
- new net: D3.2 (A), Q3.3 (E)
- new net: C8.1, Q10.2 (B)
- new net: D10.2 (A), Q10.3 (E)
- new net: Q11.1 (C), R11.2
- new net: Q18.1 (C), R18.2
- new net: Q21.1 (C), R21.2
- new net: D21.2 (A), Q21.3 (E)
- new net: C4.1, Q5.2 (B)
- new net: D5.2 (A), Q5.3 (E)
- new net: Q8.1 (C), R8.2
- new net: Q29.1 (C), R29.2
- new net: D18.2 (A), Q18.3 (E)
- new net GND: D1.1 (K), D10.1 (K), D11.1 (K), D12.1 (K), D13.1 (K), D14.1 (K), D15.1 (K), D16.1 (K), D17.1 (K), D18.1 (K), D19.1 (K), D2.1 (K), D20.1 (K), D21.1 (K), D22.1 (K), D23.1 (K), D24.1 (K), D25.1 (K), D26.1 (K), D27.1 (K), D28.1 (K), D29.1 (K), D3.1 (K), D30.1 (K), D4.1 (K), D5.1 (K), D6.1 (K), D7.1 (K), D8.1 (K), D9.1 (K)
- new net VCC: SW1.1
Other:
- title: (none) -> Fireworks PCB

Commit message: Add fabrication files and finish routing
Parts:
- removed C11, C12, C15, C16, C19, C20, C23, C24: 10u, symbol Device:C
- removed D19, D20, D24, D25, D29, D30: LED, symbol Device:LED
- removed Q19, Q20, Q24, Q25, Q29, Q30: NPN, symbol Simulation_SPICE:NPN
- removed R19, R20, R24, R25, R29, R30: 1K, symbol Device:R
- added J1: Conn_01x02, Connector_PinHeader_2.54mm:PinHeader_1x02_P2.54mm_Vertical, symbol Connector_Generic:Conn_01x02
- C1, C10, C13, C14, C17, C18, C2, C21, C22, C3, C4, C5, C6, C7, C8, C9: footprint (none) -> Connector_PinHeader_2.54mm:PinHeader_1x02_P2.54mm_Vertical
- D1, D10, D11, D12, D13, D14, D15, D16, D17, D18, D2, D21, D22, D23, D26, D27, D28, D3, D4, D5, D6, D7, D8, D9: footprint (none) -> LED_THT:LED_D5.0mm
- Q1, Q10, Q11, Q12, Q13, Q14, Q15, Q16, Q17, Q18, Q2, Q21, Q22, Q23, Q26, Q27, Q28, Q3, Q4, Q5, Q6, Q7, Q8, Q9: footprint (none) -> Package_TO_SOT_THT:TO-92L_Inline_Wide
- R1, R10, R11, R12, R13, R14, R15, R16, R17, R18, R2, R21, R22, R23, R26, R27, R28, R3, R4, R5, R6, R7, R8, R9: footprint (none) -> Resistor_THT:R_Axial_DIN0204_L3.6mm_D1.6mm_P7.62mm_Horizontal
- SW1: footprint (none) -> Button_Switch_THT:SW_PUSH_6mm
Connections:
- net GND: now also J1.2 (Pin_2)
- net VCC: now also J1.1 (Pin_1)
- net at Q4.2 (B): now also C3.2, C4.2; no longer C3.1
- net at C1.2, C2.2, Q1.2 (B): no longer C3.2, C4.2
- net at Q9.2 (B): now also C4.1; no longer C7.1
- net at C5.2, C6.2, Q6.2 (B): no longer C7.2, C8.2
- net at Q14.2 (B): now also C7.1
- net at Q15.2 (B): now also C8.1
- net at Q10.2 (B): now also C7.2, C8.2; no longer C8.1
- net at Q5.2 (B): now also C3.1; no longer C4.1
Other:
- moved on the sheet: C1, C10, C13, C14, C17, C18, C2, C21, C22, C5, C6, C9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

Commit message: Correct capacitor footprint
Parts:
- C1, C10, C13, C14, C17, C18, C2, C21, C22, C3, C4, C5, C6, C7, C8, C9: footprint Connector_PinHeader_2.54mm:PinHeader_1x02_P2.54mm_Vertical -> Capacitor_THT:C_Disc_D5.0mm_W2.5mm_P5.00mm
Changed lines of the file:
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@@
 			)
 		)
-		(property "Footprint" "Connector_PinHeader_2.54mm:PinHeader_1x02_P2.54mm_Vertical"
+		(property "Footprint" "Capacitor_THT:C_Disc_D5.0mm_W2.5mm_P5.00mm"
 			(at 153.3652 50.8 0)
 			(effects
@@
 			)
 		)
-		(property "Footprint" "Connector_PinHeader_2.54mm:PinHeader_1x02_P2.54mm_Vertical"
+		(property "Footprint" "Capacitor_THT:C_Disc_D5.0mm_W2.5mm_P5.00mm"
 			(at 127.9652 50.8 0)
 			(effects
@@
 			)
 		)
-		(property "Footprint" "Connector_PinHeader_2.54mm:PinHeader_1x02_P2.54mm_Vertical"
+		(property "Footprint" "Capacitor_THT:C_Disc_D5.0mm_W2.5mm_P5.00mm"
 			(at 153.3652 124.46 0)
 			(effects
@@
 			)
 		)
-		(property "Footprint" "Connector_PinHeader_2.54mm:PinHeader_1x02_P2.54mm_Vertical"
+		(property "Footprint" "Capacitor_THT:C_Disc_D5.0mm_W2.5mm_P5.00mm"
 			(at 270.2052 165.1 0)
 			(effects
@@
 			)
 		)
-		(property "Footprint" "Connector_PinHeader_2.54mm:PinHeader_1x02_P2.54mm_Vertical"
+		(property "Footprint" "Capacitor_THT:C_Disc_D5.0mm_W2.5mm_P5.00mm"
 			(at 153.3652 87.63 0)
 			(effects
@@
 			)
 		)
-		(property "Footprint" "Connector_PinHeader_2.54mm:PinHeader_1x02_P2.54mm_Vertical"
+		(property "Footprint" "Capacitor_THT:C_Disc_D5.0mm_W2.5mm_P5.00mm"
 			(at 270.2052 50.8 0)
 			(effects
@@
 			)
 		)
-		(property "Footprint" "Connector_PinHeader_2.54mm:PinHeader_1x02_P2.54mm_Vertical"
+		(property "Footprint" "Capacitor_THT:C_Disc_D5.0mm_W2.5mm_P5.00mm"
 			(at 295.6052 50.8 0)
 			(effects
@@
 			)
 		)
-		(property "Footprint" "Connector_PinHeader_2.54mm:PinHeader_1x02_P2.54mm_Vertical"
+		(property "Footprint" "Capacitor_THT:C_Disc_D5.0mm_W2.5mm_P5.00mm"
 			(at 271.4752 86.36 0)
 			(effects
@@
 			)
 		)
-		(property "Footprint" "Connector_PinHeader_2.54mm:PinHeader_1x02_P2.54mm_Vertical"
+		(property "Footprint" "Capacitor_THT:C_Disc_D5.0mm_W2.5mm_P5.00mm"
 			(at 295.6052 165.1 0)
 			(effects
@@
 			)
 		)
-		(property "Footprint" "Connector_PinHeader_2.54mm:PinHeader_1x02_P2.54mm_Vertical"
+		(property "Footprint" "Capacitor_THT:C_Disc_D5.0mm_W2.5mm_P5.00mm"
 			(at 295.6052 124.46 0)
 			(effects
@@
 			)
 		)
-		(property "Footprint" "Connector_PinHeader_2.54mm:PinHeader_1x02_P2.54mm_Vertical"
+		(property "Footprint" "Capacitor_THT:C_Disc_D5.0mm_W2.5mm_P5.00mm"
 			(at 127.9652 165.1 0)
 			(effects
@@
 			)
 		)
-		(property "Footprint" "Connector_PinHeader_2.54mm:PinHeader_1x02_P2.54mm_Vertical"
+		(property "Footprint" "Capacitor_THT:C_Disc_D5.0mm_W2.5mm_P5.00mm"
 			(at 153.3652 165.1 0)
 			(effects
@@
 			)
 		)
-		(property "Footprint" "Connector_PinHeader_2.54mm:PinHeader_1x02_P2.54mm_Vertical"
+		(property "Footprint" "Capacitor_THT:C_Disc_D5.0mm_W2.5mm_P5.00mm"
 			(at 270.2052 124.46 0)
 			(effects
@@
 			)
 		)
-		(property "Footprint" "Connector_PinHeader_2.54mm:PinHeader_1x02_P2.54mm_Vertical"
+		(property "Footprint" "Capacitor_THT:C_Disc_D5.0mm_W2.5mm_P5.00mm"
 			(at 127.9652 124.46 0)
 			(effects
@@
 			)
 		)
-		(property "Footprint" "Connector_PinHeader_2.54mm:PinHeader_1x02_P2.54mm_Vertical"
+		(property "Footprint" "Capacitor_THT:C_Disc_D5.0mm_W2.5mm_P5.00mm"
 			(at 127.9652 87.63 0)
 			(effects
@@
 			)
 		)
-		(property "Footprint" "Connector_PinHeader_2.54mm:PinHeader_1x02_P2.54mm_Vertical"
+		(property "Footprint" "Capacitor_THT:C_Disc_D5.0mm_W2.5mm_P5.00mm"
 			(at 296.8752 86.36 0)
 			(effects
